File: VESC_6.4.kicad_pcb (KiCad board)
At the start: 4 copper layers, 62 x 60 mm, 144 parts, among them J1 CAN, J10 SUPPLY, J11 GND, J2 HALL_ENC, J3 COMM, J4 SERVO, J5 SWD, J6 USB_OTG, J7 PH_A, J8 PH_B, J9 PH_C, Q1 IRF7749, Q2 IRF7749, Q3 IRF7749, Q4 IRF7749, Q5 IRF7749, Q6 IRF7749, SW1 SENSOR_VOLTAGE, U1 STM32F40X_LQFP64, U10 MPU9250, U2 LM3671, U3 DRV8301, U4 AD8418, U5 AD8418, U6 AD8418, U7 TJA1051TK-3, U8 NRF24L01P, U9 CONN_U.FL, Y1 Crystal_GND3, Y2 16MHz

Commit message: minor PCB work
Parts:
- moved C3 13.8 mm to (143.6, 110.5)
- moved C13 0.47 mm to (145.8, 109.8)
Routing:
- net +5V: track 6.52 -> 27.5 mm
- net /MPU9250/SCL: track 0.00 -> 16.5 mm, vias 0 -> 1
- net /MCU/RX_SDA_NSS: track 0.00 -> 16.0 mm, vias 0 -> 1
- net Net-(C54-Pad2): track 2.03 -> 15.7 mm, vias 0 -> 1
- net VCC: track 13.7 -> 25.9 mm, vias 0 -> 1
- net Net-(C5-Pad2): track 2.40 -> 14.4 mm, vias 0 -> 1
- net /MCU/AN_IN: track 0.00 -> 11.8 mm, vias 0 -> 1
- net /DRV/SENS_C: track 0.00 -> 11.3 mm, vias 0 -> 1
- net Net-(J2-Pad1): track 2.94 -> 13.2 mm, vias 0 -> 1
- net /MCU/SCK_ADC_EXT: track 0.00 -> 9.97 mm, vias 0 -> 1
- net /MCU/USB_DP: track 0.00 -> 9.01 mm, vias 0 -> 1
- net /DRV/SENS_B: track 0.00 -> 8.08 mm, vias 0 -> 1
- net Net-(J6-Pad2): track 0.00 -> 8.07 mm
- net Net-(J6-Pad3): track 0.00 -> 7.87 mm
- net /MCU/USB_DM: track 0.00 -> 7.30 mm, vias 0 -> 1
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
Commit message: lots of PCB work
Parts:
- C13: moved to B.Cu
- C43, C44: footprint Capacitors_THT:CP_Radial_D12.5mm_P5.00mm -> Global_Parts:CP_Radial_D12.5mm_P5.00mm
- moved Q1 12.0 mm to (155.2, 86.6), turned to 0 degrees
- moved Q2 12.0 mm to (155.2, 74.6), turned to 90 degrees
- moved Q3 12.0 mm to (166.7, 86.6), turned to 0 degrees
- moved Q4 12.0 mm to (166.7, 74.6), turned to 90 degrees
- moved Q5 12.0 mm to (178.2, 86.6), turned to 0 degrees
- moved Q6 12.0 mm to (178.2, 74.6), turned to 90 degrees
- moved C3 1.83 mm to (145.3, 109.8), turned to 0 degrees
- moved C13 1.50 mm to (145.9, 108.3)
- moved D5 0.33 mm to (127.1, 72.1)
- moved R6 0.29 mm to (137.6, 113.2)
- moved R5 0.29 mm to (136.1, 113.2)
- moved C31 0.27 mm to (133.5, 69.7)
- moved C29 0.24 mm to (145.4, 81.0)
- moved C43 0.10 mm to (153.5, 92.2)
- moved C44 0.10 mm to (180.0, 92.2)
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Connections:
- Q1 pad 1: Net-(Q1-Pad1) -> SUPPLY
- Q1 pad 2: /DRV/SH_A -> Net-(Q1-Pad2)
- Q1 pad 3: SUPPLY -> /DRV/SH_A
- Q2 pad 1: Net-(Q2-Pad1) -> /DRV/SH_A
- Q2 pad 2: GND -> Net-(Q2-Pad2)
- Q2 pad 3: /DRV/SH_A -> GND
- Q3 pad 1: Net-(Q3-Pad1) -> SUPPLY
- Q3 pad 2: /DRV/SH_B -> Net-(Q3-Pad2)
- Q3 pad 3: SUPPLY -> /DRV/SH_B
- Q4 pad 1: Net-(Q4-Pad1) -> /DRV/SH_B
- Q4 pad 2: GND -> Net-(Q4-Pad2)
- Q4 pad 3: /DRV/SH_B -> GND
- Q5 pad 1: Net-(Q5-Pad1) -> SUPPLY
- Q5 pad 2: /DRV/SH_C -> Net-(Q5-Pad2)
- Q5 pad 3: SUPPLY -> /DRV/SH_C
- Q6 pad 1: Net-(Q6-Pad1) -> /DRV/SH_C
- Q6 pad 2: GND -> Net-(Q6-Pad2)
- Q6 pad 3: /DRV/SH_C -> GND
- R29 pad 1: Net-(Q1-Pad1) -> Net-(Q1-Pad2)
- R30 pad 1: Net-(Q2-Pad1) -> Net-(Q2-Pad2)
- R33 pad 1: Net-(Q3-Pad1) -> Net-(Q3-Pad2)
- R34 pad 1: Net-(Q4-Pad1) -> Net-(Q4-Pad2)
- R36 pad 1: Net-(Q5-Pad1) -> Net-(Q5-Pad2)
- R37 pad 1: Net-(Q6-Pad1) -> Net-(Q6-Pad2)
- U9 pad 3: (no net) -> GND
Routing:
- net +5V: track 27.5 -> 122.1 mm, vias 0 -> 6
- net /MCU/TEMP_MOTOR: track 8.72 -> 66.4 mm, vias 0 -> 2
- net Net-(R35-Pad2): track 0.00 -> 56.8 mm, vias 0 -> 2
- net Net-(R35-Pad3): track 0.00 -> 53.0 mm, vias 0 -> 2
- net /MCU/SWDIO: track 0.00 -> 45.9 mm, vias 0 -> 2
- net VCC: track 25.9 -> 56.5 mm, vias 1 -> 19
- net Net-(R31-Pad3): track 6.86 -> 35.0 mm, vias 1 -> 2
- net Net-(R31-Pad2): track 10.1 -> 38.2 mm, vias 1 -> 2
- net GND: track 3.17 -> 30.7 mm, vias 0 -> 25
- net /MCU/CAN_TX: track 0.00 -> 25.8 mm, vias 0 -> 4
- net /MCU/SERVO: track 1.44 -> 25.9 mm, vias 0 -> 2
- net /MCU/ADC_15: track 0.00 -> 23.7 mm
- net /MCU/CAN_RX: track 0.00 -> 23.4 mm, vias 0 -> 2
- net /MCU/PB4: track 0.00 -> 21.1 mm
- net /NRF/MOSI: track 0.00 -> 20.8 mm
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- added copper zone on F.Cu, net /DRV/SH_B
- added copper zone on In2.Cu, net GND
- added copper zone on F.Cu, net SUPPLY
- added copper zone on In1.Cu, net VCC
Other:
- net class Default: clearance 0.13 -> 0
- rule trace_clearance: 0.13 -> 0

Commit message: power electronics PCB work
Routing:
- added copper zone on F.Cu, net /DRV/SH_A
- added copper zone on F.Cu, net /DRV/SH_C
- added copper zone on F.Cu, net GND
- added copper zone on B.Cu, net Net-(J7-Pad1)
- added copper zone on B.Cu, net Net-(J8-Pad1)
- added copper zone on B.Cu, net Net-(J9-Pad1)
Changed lines of the file:
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@@
-(kicad_pcb (version 20170123) (host pcbnew "(2017-08-25 revision dd37d0595)-makepkg")
+(kicad_pcb (version 4) (host pcbnew 4.0.2-stable)
   (general
+    (links 454)
+    (no_connects 211)
+    (area 121.3699 61.2254 184.782401 125.8174)
     (thickness 1.6)
     (drawings 11)
@@
       (hpglpenspeed 20)
       (hpglpendiameter 15)
+      (hpglpenoverlay 2)
       (psnegative false)
       (psa4output false)
@@
     (at 138.7983 84.8741 270)
     (attr smd)
-    (fp_text reference U3 (at -8.4 0) (layer F.SilkS)
+    (fp_text reference U3 (at -8.4 0 360) (layer F.SilkS)
       (effects (font (size 0.5 0.5) (thickness 0.125)))
     )
@@
     (tags "capacitor 0603")
     (attr smd)
-    (fp_text reference C55 (at 1.75115 0.00898 45) (layer F.SilkS)
+    (fp_text reference C55 (at 1.75115 0.00898 405) (layer F.SilkS)
       (effects (font (size 0.5 0.5) (thickness 0.125)))
     )
@@
     (tags "resistor 0603")
     (attr smd)
-    (fp_text reference R29 (at -1.651 -0.0254 90) (layer B.SilkS)
+    (fp_text reference R29 (at -1.651 -0.0254 450) (layer B.SilkS)
       (effects (font (size 0.5 0.5) (thickness 0.125)) (justify mirror))
     )
-    (fp_text value 4.7 (at 1.5875 -0.0254 90) (layer B.Fab)
+    (fp_text value 4.7 (at 1.5875 -0.0254 450) (layer B.Fab)
       (effects (font (size 0.5 0.5) (thickness 0.125)) (justify mirror))
     )
@@
     (tags "resistor 0603")
     (attr smd)
-    (fp_text reference R30 (at -1.6764 -0.0127 90) (layer B.SilkS)
+    (fp_text reference R30 (at -1.6764 -0.0127 450) (layer B.SilkS)
       (effects (font (size 0.5 0.5) (thickness 0.125)) (justify mirror))
     )
-    (fp_text value 4.7 (at 1.6002 0 90) (layer B.Fab)
+    (fp_text value 4.7 (at 1.6002 0 450) (layer B.Fab)
       (effects (font (size 0.5 0.5) (thickness 0.125)) (justify mirror))
     )
@@
     (tags "resistor 0603")
     (attr smd)
-    (fp_text reference R33 (at -1.6637 0 90) (layer B.SilkS)
+    (fp_text reference R33 (at -1.6637 0 450) (layer B.SilkS)
       (effects (font (size 0.5 0.5) (thickness 0.125)) (justify mirror))
     )
-    (fp_text value 4.7 (at 1.6256 -0.0127 90) (layer B.Fab)
+    (fp_text value 4.7 (at 1.6256 -0.0127 450) (layer B.Fab)
       (effects (font (size 0.5 0.5) (thickness 0.125)) (justify mirror))
     )
@@
     (tags "resistor 0603")
     (attr smd)
-    (fp_text reference R34 (at -1.6764 0 90) (layer B.SilkS)
+    (fp_text reference R34 (at -1.6764 0 450) (layer B.SilkS)
       (effects (font (size 0.5 0.5) (thickness 0.125)) (justify mirror))
     )
-    (fp_text value 4.7 (at 1.6256 -0.0127 90) (layer B.Fab)
+    (fp_text value 4.7 (at 1.6256 -0.0127 450) (layer B.Fab)
       (effects (font (size 0.5 0.5) (thickness 0.125)) (justify mirror))
     )
@@
     (tags "resistor 0603")
     (attr smd)
-    (fp_text reference R36 (at -1.651 0 90) (layer B.SilkS)
+    (fp_text reference R36 (at -1.651 0 450) (layer B.SilkS)
       (effects (font (size 0.5 0.5) (thickness 0.125)) (justify mirror))
     )
-    (fp_text value 4.7 (at 1.6002 -0.0381 90) (layer B.Fab)
+    (fp_text value 4.7 (at 1.6002 -0.0381 450) (layer B.Fab)
       (effects (font (size 0.5 0.5) (thickness 0.125)) (justify mirror))
     )
@@
     (tags "resistor 0603")
     (attr smd)
-    (fp_text reference R37 (at 1.6637 -0.0127 90) (layer B.SilkS)
+    (fp_text reference R37 (at 1.6637 -0.0127 450) (layer B.SilkS)
       (effects (font (size 0.5 0.5) (thickness 0.125)) (justify mirror))
     )
-    (fp_text value 4.7 (at -1.6383 -0.0127 90) (layer B.Fab)
+    (fp_text value 4.7 (at -1.6383 -0.0127 450) (layer B.Fab)
       (effects (font (size 0.5 0.5) (thickness 0.125)) (justify mirror))
     )
@@
       (effects (font (size 0.5 0.5) (thickness 0.125)))
     )
-    (fp_text value NRF24L01P (at 7.830783 -8.046309 45) (layer F.Fab)
+    (fp_text value NRF24L01P (at 7.830783 -8.046309 405) (layer F.Fab)
       (effects (font (size 0.5 0.5) (thickness 0.125)))
     )
@@
     (fp_line (start 0.9 1.61) (end -1.55 1.61) (layer B.SilkS) (width 0.12))
     (fp_line (start -0.9 -1.61) (end 0.9 -1.61) (layer B.SilkS) (width 0.12))
-    (fp_text user %R (at 0 0 90) (layer B.Fab)
+    (fp_text user %R (at 0 0 450) (layer B.Fab)
       (effects (font (size 0.5 0.5) (thickness 0.125)) (justify mirror))
     )
@@
     )
   )
+  (zone (net 25) (net_name /DRV/SH_C) (layer F.Cu) (hatch edge 0.508)
+    (connect_pads yes (clearance 0.1))
+    (min_thickness 0.254)
+    (fill yes (arc_segments 16) (thermal_gap 0.508) (thermal_bridge_width 0.508))
+    (polygon
+      (pts
+        (xy 181.483 78.486) (xy 181.483 83.058) (xy 181.229 83.312) (xy 181.229 89.154) (xy 176.403 89.154)
+        (xy 176.403 88.4301) (xy 176.403 83.185) (xy 176.149 82.931) (xy 175.133 82.931) (xy 174.879 82.677)
+        (xy 174.879 78.486)
+      )
+    )
+  )
+  (zone (net 21) (net_name /DRV/SH_A) (layer F.Cu) (hatch edge 0.508)
+    (connect_pads yes (clearance 0.1))
+    (min_thickness 0.254)
+    (fill yes (arc_segments 16) (thermal_gap 0.508) (thermal_bridge_width 0.508))
+    (polygon
+      (pts
+        (xy 158.496 78.484748) (xy 158.496 83.056748) (xy 158.242 83.310748) (xy 158.242 89.152748) (xy 153.416 89.152748)
+        (xy 153.416 88.428848) (xy 153.416 83.183748) (xy 153.162 82.929748) (xy 152.146 82.929748) (xy 151.892 82.675748)
+        (xy 151.892 78.484748)
+      )
+    )
+  )
   (zone (net 22) (net_name /DRV/SH_B) (layer F.Cu) (hatch edge 0.508)
     (connect_pads yes (clearance 0.1))
-    (min_thickness 1)
+    (min_thickness 0.254)
+    (fill yes (arc_segments 16) (thermal_gap 0.508) (thermal_bridge_width 0.508))
+    (polygon
+      (pts
+        (xy 170.053 78.484748) (xy 170.053 83.056748) (xy 169.799 83.310748) (xy 169.799 89.152748) (xy 164.973 89.152748)
+        (xy 164.973 88.428848) (xy 164.973 83.183748) (xy 164.719 82.929748) (xy 163.703 82.929748) (xy 163.449 82.675748)
+        (xy 163.449 78.484748)
+      )
+    )
+  )
+  (zone (net 2) (net_name GND) (layer F.Cu) (hatch edge 0.508)
+    (connect_pads yes (clearance 0.1))
+    (min_thickness 0.254)
+    (fill yes (arc_segments 16) (thermal_gap 0.508) (thermal_bridge_width 0.508))
+    (polygon
+      (pts
+        (xy 181.356 76.327) (xy 181.356 71.628) (xy 152.019 71.628) (xy 152.019 76.3905) (xy 159.131 76.3905)
+        (xy 159.131 77.597) (xy 162.814 77.597) (xy 162.814 76.5175) (xy 162.814 76.3905) (xy 170.561 76.3905)
+        (xy 170.561 77.597) (xy 174.371 77.597) (xy 174.371 76.3905) (xy 181.356 76.4032)
+      )
+    )
+  )
+  (zone (net 137) (net_name "Net-(J8-Pad1)") (layer B.Cu) (hatch edge 0.508)
+    (connect_pads yes (clearance 0.1))
+    (min_thickness 0.254)
+    (fill yes (arc_segments 16) (thermal_gap 0.508) (thermal_bridge_width 0.508))
+    (polygon
+      (pts
+        (xy 163.576 73.3044) (xy 163.576 70.485) (xy 163.576 64.77) (xy 169.799 64.77) (xy 169.8371 64.77)
+        (xy 169.8371 73.3044)
+      )
+    )
+  )
+  (zone (net 136) (net_name "Net-(J7-Pad1)") (layer B.Cu) (hatch edge 0.508)
+    (connect_pads yes (clearance 0.1))
+    (min_thickness 0.254)
+    (fill yes (arc_segments 16) (thermal_gap 0.508) (thermal_bridge_width 0.508))
+    (polygon
+      (pts
+        (xy 163.5633 73.279003) (xy 163.5633 70.459603) (xy 163.5633 64.744603) (xy 169.7863 64.744603) (xy 169.8244 64.744603)
+        (xy 169.8244 73.279003)
+      )
+    )
+  )
+  (zone (net 138) (net_name "Net-(J9-Pad1)") (layer B.Cu) (hatch edge 0.508)
+    (connect_pads yes (clearance 0.1))
+    (min_thickness 0.254)
     (fill yes (arc_segments 16) (thermal_gap 0.508) (thermal_bridge_width 0.508))
     (polygon
       (pts
-        (xy 169.9641 78.4987) (xy 169.9641 88.2142) (xy 169.9641 89.027) (xy 164.8587 89.027) (xy 164.8587 84.201)
-        (xy 163.322 84.201) (xy 163.322 78.486) (xy 169.9641 78.486)
+        (xy 163.5633 73.286983) (xy 163.5633 70.467583) (xy 163.5633 64.752583) (xy 169.7863 64.752583) (xy 169.8244 64.752583)
+        (xy 169.8244 73.286983)
       )
     )

Commit message: Continued Work on the PCB
Parts:
- moved C7 1.13 mm to (139.8, 98.9), turned to 90 degrees
- moved C43 0.30 mm to (153.5, 92.5)
- moved C44 0.30 mm to (180.0, 92.5)
Routing:
- net /MCU/NRST: track 3.94 -> 37.1 mm
- net /MCU/MISO_ADC_EXT2: track 0.00 -> 18.4 mm, vias 0 -> 1
- net GND: track 30.7 -> 36.9 mm, vias 25 -> 27
- net VCC: track 56.5 -> 59.4 mm, vias 19 -> 22
- net Net-(R31-Pad2): track 38.2 -> 40.0 mm
- net /MCU/SWDIO: track 45.9 -> 45.0 mm
- added copper zone on B.Cu, net /DRV/SH_A
- added copper zone on B.Cu, net /DRV/SH_B
- added copper zone on B.Cu, net /DRV/SH_C
- added copper zone on B.Cu, net GND

Commit message: power electronics almost done
Parts:
- added ?: , Global_Parts:via-0.45mm, F.Cu at (180.3, 68.0)
- added ?: , Global_Parts:via-0.45mm, F.Cu at (178.9, 67.3)
- added ?: , Global_Parts:via-0.45mm, F.Cu at (168.1, 65.2)
- added ?: , Global_Parts:via-0.45mm, F.Cu at (167.4, 65.2)
- added ?: , Global_Parts:via-0.45mm, F.Cu at (166.7, 65.2)
- added ?: , Global_Parts:via-0.45mm, F.Cu at (166.0, 65.2)
- added ?: , Global_Parts:via-0.45mm, F.Cu at (165.3, 65.2)
- added ?: , Global_Parts:via-0.45mm, F.Cu at (164.6, 65.2)
- added ?: , Global_Parts:via-0.45mm, F.Cu at (162.0, 76.8)
- added ?: , Global_Parts:via-0.45mm, F.Cu at (161.3, 76.1)
- added ?: , Global_Parts:via-0.45mm, F.Cu at (162.0, 74.7)
- added ?: , Global_Parts:via-0.45mm, F.Cu at (161.3, 76.8)
- added ?: , Global_Parts:via-0.45mm, F.Cu at (178.2, 67.3)
- added ?: , Global_Parts:via-0.45mm, F.Cu at (162.0, 72.6)
- added ?: , Global_Parts:via-0.45mm, F.Cu at (160.6, 76.1)
- added ?: , Global_Parts:via-0.45mm, F.Cu at (160.6, 76.8)
- added ?: , Global_Parts:via-0.45mm, F.Cu at (160.6, 75.4)
- added ?: , Global_Parts:via-0.45mm, F.Cu at (160.6, 74.0)
- added ?: , Global_Parts:via-0.45mm, F.Cu at (159.9, 74.7)
- added ?: , Global_Parts:via-0.45mm, F.Cu at (162.0, 74.0)
- added ?: , Global_Parts:via-0.45mm, F.Cu at (159.9, 76.1)
- added ?: , Global_Parts:via-0.45mm, F.Cu at (161.3, 75.4)
- added ?: , Global_Parts:via-0.45mm, F.Cu at (161.3, 74.7)
- added ?: , Global_Parts:via-0.45mm, F.Cu at (177.5, 67.3)
- added ?: , Global_Parts:via-0.45mm, F.Cu at (159.9, 76.8)
- added ?: , Global_Parts:via-0.45mm, F.Cu at (160.6, 72.6)
- added ?: , Global_Parts:via-0.45mm, F.Cu at (161.3, 73.3)
- added ?: , Global_Parts:via-0.45mm, F.Cu at (159.9, 75.4)
- added ?: , Global_Parts:via-0.45mm, F.Cu at (162.0, 76.1)
- added ?: , Global_Parts:via-0.45mm, F.Cu at (161.3, 74.0)
- added ?: , Global_Parts:via-0.45mm, F.Cu at (162.0, 73.3)
- added ?: , Global_Parts:via-0.45mm, F.Cu at (159.9, 72.6)
- added ?: , Global_Parts:via-0.45mm, F.Cu at (162.0, 75.4)
- added ?: , Global_Parts:via-0.45mm, F.Cu at (160.6, 74.7)
- added ?: , Global_Parts:via-0.45mm, F.Cu at (176.8, 67.3)
- added ?: , Global_Parts:via-0.45mm, F.Cu at (159.9, 74.0)
- added ?: , Global_Parts:via-0.45mm, F.Cu at (160.6, 73.3)
- added ?: , Global_Parts:via-0.45mm, F.Cu at (161.3, 72.6)
- added ?: , Global_Parts:via-0.45mm, F.Cu at (159.9, 73.3)
- added ?: , Global_Parts:via-0.45mm, F.Cu at (173.5, 76.8)
- added ?: , Global_Parts:via-0.45mm, F.Cu at (172.8, 76.8)
- added ?: , Global_Parts:via-0.45mm, F.Cu at (172.1, 76.8)
- added ?: , Global_Parts:via-0.45mm, F.Cu at (171.4, 76.8)
- added ?: , Global_Parts:via-0.45mm, F.Cu at (173.5, 76.1)
- added ?: , Global_Parts:via-0.45mm, F.Cu at (172.8, 76.1)
- added ?: , Global_Parts:via-0.45mm, F.Cu at (176.1, 67.3)
- added ?: , Global_Parts:via-0.45mm, F.Cu at (172.1, 76.1)
- added ?: , Global_Parts:via-0.45mm, F.Cu at (171.4, 76.1)
- added ?: , Global_Parts:via-0.45mm, F.Cu at (173.5, 75.4)
- added ?: , Global_Parts:via-0.45mm, F.Cu at (172.8, 75.4)
- added ?: , Global_Parts:via-0.45mm, F.Cu at (172.1, 75.4)
- added ?: , Global_Parts:via-0.45mm, F.Cu at (171.4, 75.4)
- added ?: , Global_Parts:via-0.45mm, F.Cu at (173.5, 74.7)
- added ?: , Global_Parts:via-0.45mm, F.Cu at (172.8, 74.7)
- added ?: , Global_Parts:via-0.45mm, F.Cu at (172.1, 74.7)
- added ?: , Global_Parts:via-0.45mm, F.Cu at (171.4, 74.7)
- added ?: , Global_Parts:via-0.45mm, F.Cu at (180.3, 66.6)
- added ?: , Global_Parts:via-0.45mm, F.Cu at (173.5, 74.0)
- added ?: , Global_Parts:via-0.45mm, F.Cu at (172.8, 74.0)
- added ?: , Global_Parts:via-0.45mm, F.Cu at (172.1, 74.0)
- added ?: , Global_Parts:via-0.45mm, F.Cu at (171.4, 74.0)
- added ?: , Global_Parts:via-0.45mm, F.Cu at (173.5, 73.3)
- added ?: , Global_Parts:via-0.45mm, F.Cu at (172.8, 73.3)
- added ?: , Global_Parts:via-0.45mm, F.Cu at (172.1, 73.3)
- added ?: , Global_Parts:via-0.45mm, F.Cu at (171.4, 73.3)
- added ?: , Global_Parts:via-0.45mm, F.Cu at (173.5, 72.6)
- added ?: , Global_Parts:via-0.45mm, F.Cu at (172.8, 72.6)
- added ?: , Global_Parts:via-0.45mm, F.Cu at (179.6, 66.6)
- added ?: , Global_Parts:via-0.45mm, F.Cu at (172.1, 72.6)
- added ?: , Global_Parts:via-0.45mm, F.Cu at (171.4, 72.6)
- added ?: , Global_Parts:via-0.45mm, F.Cu at (157.3, 84.2)
- added ?: , Global_Parts:via-0.45mm, F.Cu at (156.6, 84.2)
- added ?: , Global_Parts:via-0.45mm, F.Cu at (155.9, 84.2)
- added ?: , Global_Parts:via-0.45mm, F.Cu at (155.2, 84.2)
- added ?: , Global_Parts:via-0.45mm, F.Cu at (154.5, 84.2)
- added ?: , Global_Parts:via-0.45mm, F.Cu at (153.8, 84.2)
- added ?: , Global_Parts:via-0.45mm, F.Cu at (153.1, 84.2)
- added ?: , Global_Parts:via-0.45mm, F.Cu at (157.3, 83.5)
- added ?: , Global_Parts:via-0.45mm, F.Cu at (178.9, 66.6)
- added ?: , Global_Parts:via-0.45mm, F.Cu at (156.6, 83.5)
- added ?: , Global_Parts:via-0.45mm, F.Cu at (155.9, 83.5)
- added ?: , Global_Parts:via-0.45mm, F.Cu at (155.2, 83.5)
- added ?: , Global_Parts:via-0.45mm, F.Cu at (154.5, 83.5)
- added ?: , Global_Parts:via-0.45mm, F.Cu at (153.8, 83.5)
- added ?: , Global_Parts:via-0.45mm, F.Cu at (153.1, 83.5)
- added ?: , Global_Parts:via-0.45mm, F.Cu at (157.3, 82.8)
- added ?: , Global_Parts:via-0.45mm, F.Cu at (156.6, 82.8)
- added ?: , Global_Parts:via-0.45mm, F.Cu at (155.9, 82.8)
- added ?: , Global_Parts:via-0.45mm, F.Cu at (155.2, 82.8)
- added ?: , Global_Parts:via-0.45mm, F.Cu at (178.2, 66.6)
- added ?: , Global_Parts:via-0.45mm, F.Cu at (154.5, 82.8)
- added ?: , Global_Parts:via-0.45mm, F.Cu at (153.8, 82.8)
- added ?: , Global_Parts:via-0.45mm, F.Cu at (153.1, 82.8)
- added ?: , Global_Parts:via-0.45mm, F.Cu at (157.3, 82.1)
- added ?: , Global_Parts:via-0.45mm, F.Cu at (156.6, 82.1)
- added ?: , Global_Parts:via-0.45mm, F.Cu at (155.9, 82.1)
- added ?: , Global_Parts:via-0.45mm, F.Cu at (155.2, 82.1)
- added ?: , Global_Parts:via-0.45mm, F.Cu at (154.5, 82.1)
- added ?: , Global_Parts:via-0.45mm, F.Cu at (153.8, 82.1)
- added ?: , Global_Parts:via-0.45mm, F.Cu at (168.9, 84.2)
- added ?: , Global_Parts:via-0.45mm, F.Cu at (177.5, 66.6)
- added ?: , Global_Parts:via-0.45mm, F.Cu at (168.2, 84.2)
- added ?: , Global_Parts:via-0.45mm, F.Cu at (167.5, 84.2)
- added ?: , Global_Parts:via-0.45mm, F.Cu at (166.8, 84.2)
- added ?: , Global_Parts:via-0.45mm, F.Cu at (166.1, 84.2)
- added ?: , Global_Parts:via-0.45mm, F.Cu at (165.4, 84.2)
- added ?: , Global_Parts:via-0.45mm, F.Cu at (164.7, 84.2)
- added ?: , Global_Parts:via-0.45mm, F.Cu at (168.9, 83.5)
- added ?: , Global_Parts:via-0.45mm, F.Cu at (168.2, 83.5)
- added ?: , Global_Parts:via-0.45mm, F.Cu at (167.5, 83.5)
- added ?: , Global_Parts:via-0.45mm, F.Cu at (166.8, 83.5)
- added ?: , Global_Parts:via-0.45mm, F.Cu at (179.6, 68.0)
- added ?: , Global_Parts:via-0.45mm, F.Cu at (176.8, 66.6)
- added ?: , Global_Parts:via-0.45mm, F.Cu at (166.1, 83.5)
- added ?: , Global_Parts:via-0.45mm, F.Cu at (165.4, 83.5)
- added ?: , Global_Parts:via-0.45mm, F.Cu at (164.7, 83.5)
- added ?: , Global_Parts:via-0.45mm, F.Cu at (168.9, 82.8)
- added ?: , Global_Parts:via-0.45mm, F.Cu at (168.2, 82.8)
- added ?: , Global_Parts:via-0.45mm, F.Cu at (167.5, 82.8)
- added ?: , Global_Parts:via-0.45mm, F.Cu at (166.8, 82.8)
- added ?: , Global_Parts:via-0.45mm, F.Cu at (166.1, 82.8)
- added ?: , Global_Parts:via-0.45mm, F.Cu at (165.4, 82.8)
- added ?: , Global_Parts:via-0.45mm, F.Cu at (164.7, 82.8)
- added ?: , Global_Parts:via-0.45mm, F.Cu at (176.1, 66.6)
- added ?: , Global_Parts:via-0.45mm, F.Cu at (168.9, 82.1)
- added ?: , Global_Parts:via-0.45mm, F.Cu at (168.2, 82.1)
- added ?: , Global_Parts:via-0.45mm, F.Cu at (167.5, 82.1)
- added ?: , Global_Parts:via-0.45mm, F.Cu at (166.8, 82.1)
- added ?: , Global_Parts:via-0.45mm, F.Cu at (166.1, 82.1)
- added ?: , Global_Parts:via-0.45mm, F.Cu at (165.4, 82.1)
- added ?: , Global_Parts:via-0.45mm, F.Cu at (153.1, 82.1)
- added ?: , Global_Parts:via-0.45mm, F.Cu at (164.7, 82.1)
- added ?: , Global_Parts:via-0.45mm, F.Cu at (180.3, 84.2)
- added ?: , Global_Parts:via-0.45mm, F.Cu at (179.6, 84.2)
- added ?: , Global_Parts:via-0.45mm, F.Cu at (180.3, 65.9)
- added ?: , Global_Parts:via-0.45mm, F.Cu at (178.9, 84.2)
- added ?: , Global_Parts:via-0.45mm, F.Cu at (178.2, 84.2)
- added ?: , Global_Parts:via-0.45mm, F.Cu at (177.5, 84.2)
- added ?: , Global_Parts:via-0.45mm, F.Cu at (176.8, 84.2)
- added ?: , Global_Parts:via-0.45mm, F.Cu at (176.1, 84.2)
- added ?: , Global_Parts:via-0.45mm, F.Cu at (180.3, 83.5)
- added ?: , Global_Parts:via-0.45mm, F.Cu at (179.6, 83.5)
- added ?: , Global_Parts:via-0.45mm, F.Cu at (178.9, 83.5)
- added ?: , Global_Parts:via-0.45mm, F.Cu at (178.2, 83.5)
- added ?: , Global_Parts:via-0.45mm, F.Cu at (177.5, 83.5)
- added ?: , Global_Parts:via-0.45mm, F.Cu at (179.6, 65.9)
- added ?: , Global_Parts:via-0.45mm, F.Cu at (176.8, 83.5)
- added ?: , Global_Parts:via-0.45mm, F.Cu at (176.1, 83.5)
- added ?: , Global_Parts:via-0.45mm, F.Cu at (180.3, 82.8)
- added ?: , Global_Parts:via-0.45mm, F.Cu at (179.6, 82.8)
- added ?: , Global_Parts:via-0.45mm, F.Cu at (178.9, 82.8)
- added ?: , Global_Parts:via-0.45mm, F.Cu at (178.2, 82.8)
- added ?: , Global_Parts:via-0.45mm, F.Cu at (177.5, 82.8)
- added ?: , Global_Parts:via-0.45mm, F.Cu at (176.8, 82.8)
- added ?: , Global_Parts:via-0.45mm, F.Cu at (176.1, 82.8)
- added ?: , Global_Parts:via-0.45mm, F.Cu at (180.3, 82.1)
- added ?: , Global_Parts:via-0.45mm, F.Cu at (178.9, 65.9)
- added ?: , Global_Parts:via-0.45mm, F.Cu at (179.6, 82.1)
- added ?: , Global_Parts:via-0.45mm, F.Cu at (178.9, 82.1)
- added ?: , Global_Parts:via-0.45mm, F.Cu at (178.2, 82.1)
- added ?: , Global_Parts:via-0.45mm, F.Cu at (177.5, 82.1)
- added ?: , Global_Parts:via-0.45mm, F.Cu at (176.8, 82.1)
- added ?: , Global_Parts:via-0.45mm, F.Cu at (176.1, 82.1)
- added ?: , Global_Parts:via-0.45mm, F.Cu at (178.2, 65.9)
- added ?: , Global_Parts:via-0.45mm, F.Cu at (177.5, 65.9)
- added ?: , Global_Parts:via-0.45mm, F.Cu at (176.8, 65.9)
- added ?: , Global_Parts:via-0.45mm, F.Cu at (176.1, 65.9)
- added ?: , Global_Parts:via-0.45mm, F.Cu at (180.3, 65.2)
- added ?: , Global_Parts:via-0.45mm, F.Cu at (178.9, 68.0)
- added ?: , Global_Parts:via-0.45mm, F.Cu at (179.6, 65.2)
- added ?: , Global_Parts:via-0.45mm, F.Cu at (178.9, 65.2)
- added ?: , Global_Parts:via-0.45mm, F.Cu at (178.2, 65.2)
- added ?: , Global_Parts:via-0.45mm, F.Cu at (177.5, 65.2)
- added ?: , Global_Parts:via-0.45mm, F.Cu at (176.8, 65.2)
- added ?: , Global_Parts:via-0.45mm, F.Cu at (157.3, 68.0)
- added ?: , Global_Parts:via-0.45mm, F.Cu at (156.6, 68.0)
- added ?: , Global_Parts:via-0.45mm, F.Cu at (155.9, 68.0)
- added ?: , Global_Parts:via-0.45mm, F.Cu at (155.2, 68.0)
- added ?: , Global_Parts:via-0.45mm, F.Cu at (154.5, 68.0)
- added ?: , Global_Parts:via-0.45mm, F.Cu at (178.2, 68.0)
- added ?: , Global_Parts:via-0.45mm, F.Cu at (153.8, 68.0)
- added ?: , Global_Parts:via-0.45mm, F.Cu at (153.1, 68.0)
- added ?: , Global_Parts:via-0.45mm, F.Cu at (157.3, 67.3)
- added ?: , Global_Parts:via-0.45mm, F.Cu at (156.6, 67.3)
- added ?: , Global_Parts:via-0.45mm, F.Cu at (155.9, 67.3)
- added ?: , Global_Parts:via-0.45mm, F.Cu at (155.2, 67.3)
- added ?: , Global_Parts:via-0.45mm, F.Cu at (154.5, 67.3)
- added ?: , Global_Parts:via-0.45mm, F.Cu at (153.8, 67.3)
- added ?: , Global_Parts:via-0.45mm, F.Cu at (153.1, 67.3)
- added ?: , Global_Parts:via-0.45mm, F.Cu at (157.3, 66.6)
- added ?: , Global_Parts:via-0.45mm, F.Cu at (177.5, 68.0)
- added ?: , Global_Parts:via-0.45mm, F.Cu at (156.6, 66.6)
- added ?: , Global_Parts:via-0.45mm, F.Cu at (155.9, 66.6)
- added ?: , Global_Parts:via-0.45mm, F.Cu at (155.2, 66.6)
- added ?: , Global_Parts:via-0.45mm, F.Cu at (154.5, 66.6)
- added ?: , Global_Parts:via-0.45mm, F.Cu at (153.8, 66.6)
- added ?: , Global_Parts:via-0.45mm, F.Cu at (153.1, 66.6)
- added ?: , Global_Parts:via-0.45mm, F.Cu at (157.3, 65.9)
- added ?: , Global_Parts:via-0.45mm, F.Cu at (156.6, 65.9)
- added ?: , Global_Parts:via-0.45mm, F.Cu at (155.9, 65.9)
- added ?: , Global_Parts:via-0.45mm, F.Cu at (155.2, 65.9)
- added ?: , Global_Parts:via-0.45mm, F.Cu at (176.8, 68.0)
- added ?: , Global_Parts:via-0.45mm, F.Cu at (154.5, 65.9)
- added ?: , Global_Parts:via-0.45mm, F.Cu at (153.8, 65.9)
- added ?: , Global_Parts:via-0.45mm, F.Cu at (153.1, 65.9)
- added ?: , Global_Parts:via-0.45mm, F.Cu at (157.3, 65.2)
- added ?: , Global_Parts:via-0.45mm, F.Cu at (156.6, 65.2)
- added ?: , Global_Parts:via-0.45mm, F.Cu at (155.9, 65.2)
- added ?: , Global_Parts:via-0.45mm, F.Cu at (155.2, 65.2)
- added ?: , Global_Parts:via-0.45mm, F.Cu at (154.5, 65.2)
- added ?: , Global_Parts:via-0.45mm, F.Cu at (153.8, 65.2)
- added ?: , Global_Parts:via-0.45mm, F.Cu at (176.1, 65.2)
- added ?: , Global_Parts:via-0.45mm, F.Cu at (176.1, 68.0)
- added ?: , Global_Parts:via-0.45mm, F.Cu at (153.1, 65.2)
- added ?: , Global_Parts:via-0.45mm, F.Cu at (168.8, 68.0)
- added ?: , Global_Parts:via-0.45mm, F.Cu at (168.1, 68.0)
- added ?: , Global_Parts:via-0.45mm, F.Cu at (167.4, 68.0)
- added ?: , Global_Parts:via-0.45mm, F.Cu at (166.7, 68.0)
- added ?: , Global_Parts:via-0.45mm, F.Cu at (166.0, 68.0)
- added ?: , Global_Parts:via-0.45mm, F.Cu at (165.3, 68.0)
- added ?: , Global_Parts:via-0.45mm, F.Cu at (164.6, 68.0)
- added ?: , Global_Parts:via-0.45mm, F.Cu at (168.8, 67.3)
- added ?: , Global_Parts:via-0.45mm, F.Cu at (168.1, 67.3)
- added ?: , Global_Parts:via-0.45mm, F.Cu at (180.3, 67.3)
- added ?: , Global_Parts:via-0.45mm, F.Cu at (167.4, 67.3)
- added ?: , Global_Parts:via-0.45mm, F.Cu at (166.7, 67.3)
- added ?: , Global_Parts:via-0.45mm, F.Cu at (166.0, 67.3)
- added ?: , Global_Parts:via-0.45mm, F.Cu at (165.3, 67.3)
- added ?: , Global_Parts:via-0.45mm, F.Cu at (164.6, 67.3)
- added ?: , Global_Parts:via-0.45mm, F.Cu at (168.8, 66.6)
- added ?: , Global_Parts:via-0.45mm, F.Cu at (168.1, 66.6)
- added ?: , Global_Parts:via-0.45mm, F.Cu at (167.4, 66.6)
- added ?: , Global_Parts:via-0.45mm, F.Cu at (166.7, 66.6)
- added ?: , Global_Parts:via-0.45mm, F.Cu at (166.0, 66.6)
- added ?: , Global_Parts:via-0.45mm, F.Cu at (179.6, 67.3)
- added ?: , Global_Parts:via-0.45mm, F.Cu at (165.3, 66.6)
- added ?: , Global_Parts:via-0.45mm, F.Cu at (164.6, 66.6)
- added ?: , Global_Parts:via-0.45mm, F.Cu at (168.8, 65.9)
- added ?: , Global_Parts:via-0.45mm, F.Cu at (168.1, 65.9)
- added ?: , Global_Parts:via-0.45mm, F.Cu at (167.4, 65.9)
- added ?: , Global_Parts:via-0.45mm, F.Cu at (166.7, 65.9)
- added ?: , Global_Parts:via-0.45mm, F.Cu at (166.0, 65.9)
- added ?: , Global_Parts:via-0.45mm, F.Cu at (165.3, 65.9)
- added ?: , Global_Parts:via-0.45mm, F.Cu at (164.6, 65.9)
- added ?: , Global_Parts:via-0.45mm, F.Cu at (168.8, 65.2)
Routing:
- net SUPPLY: track 0.00 -> 54.8 mm, vias 0 -> 60
- net Net-(Q6-Pad2): track 0.00 -> 41.3 mm, vias 0 -> 2
- net Net-(Q5-Pad2): track 0.00 -> 33.2 mm, vias 0 -> 2
- net Net-(Q4-Pad2): track 0.00 -> 27.0 mm, vias 0 -> 2
- net Net-(Q3-Pad2): track 0.00 -> 18.6 mm, vias 0 -> 2
- net Net-(Q2-Pad2): track 0.00 -> 13.0 mm, vias 0 -> 2
- net Net-(Q1-Pad2): track 0.00 -> 8.93 mm, vias 0 -> 1
- net +5V: track 122.3 -> 125.2 mm
- net Net-(R31-Pad2): track 40.0 -> 38.7 mm
- added copper zone on F.Cu, net Net-(J7-Pad1)
- added copper zone on F.Cu, net Net-(J8-Pad1)
- added copper zone on F.Cu, net Net-(J9-Pad1)
- added copper zone on B.Cu, net SUPPLY
Other:
- net class Default: clearance 0 -> 0.13
- rule trace_clearance: 0 -> 0.13
- rule trace_min: 0.2 -> 0.13

Commit message: its a dark and scary night in kicad land
Routing:
- net /MCU/SWCLK: track 0.00 -> 48.3 mm, vias 0 -> 1
- net /MCU/TEMP_MOTOR: track 66.4 -> 65.6 mm

Commit message: the PCB trace gremlins were creeping around
Routing:
- net /DRV/SH_C: track 8.62 -> 40.7 mm, vias 1 -> 2
- net /DRV/SH_B: track 11.1 -> 30.5 mm, vias 1 -> 2
- net /DRV/INL_C: track 9.98 -> 24.8 mm, vias 0 -> 2
- net /DRV/INL_A: track 9.81 -> 24.2 mm
- net /DRV/INL_B: track 9.88 -> 23.1 mm, vias 0 -> 2
- net /DRV/SH_A: track 16.0 -> 23.5 mm, vias 1 -> 2
- net Net-(Q5-Pad2): track 33.2 -> 30.4 mm
- net /DRV/SENS_A: track 5.65 -> 7.42 mm
- net Net-(Q3-Pad2): track 18.6 -> 20.1 mm
- net Net-(Q1-Pad2): track 8.93 -> 8.18 mm
- net /DRV/SENS_C: track 11.3 -> 10.6 mm

Commit message: the save button tried its hardest to stay safe from the gremlins
Routing:
- net Net-(C29-Pad1): track 3.60 -> 11.9 mm
- net /MCU/ADC_TEMP: track 3.45 -> 8.85 mm
- net SUPPLY: track 54.8 -> 59.1 mm
- added copper zone on F.Cu, net Net-(C29-Pad1)
