File: VESC_6.4.sch (KiCad schematic (older format))
At the start: 23 parts, among them J1 CAN, J2 HALL_ENC, J3 COMM, J4 SERVO, J5 SWD, J6 USB_OTG, SW1 SENSOR_VOLTAGE

Commit message: trying out a new PCB shape, trimmed away NRF and MPU
Connections:
- no-connect marks 2 -> 1
Changed lines of the file:
@@
 $Descr A4 11693 8268
 encoding utf-8
-Sheet 1 7
+Sheet 1 5
 Title "VESC 6.4 "
 Date "2018-02-05"
@@
 Wire Wire Line
 	7150 5650 6850 5650
-$Sheet
-S 7550 4600 800  650
-U 5A7B10DC
-F0 "NRF" 60
-F1 "NRF.sch" 60
-F2 "CE" I L 7550 4700 60
-F3 "CSN" I L 7550 5100 60
-F4 "SCK" I L 7550 5000 60
-F5 "MOSI" I L 7550 4900 60
-F6 "MISO" I L 7550 4800 60
-F7 "IRQ" I R 8350 5100 60
-$EndSheet
-$Comp
-L VCC #PWR022
-U 1 1 5A7B1506
-P 7500 4700
-F 0 "#PWR022" H 7500 4550 50  0001 C CNN
-F 1 "VCC" V 7518 4827 50  0000 L CNN
-F 2 "" H 7500 4700 50  0001 C CNN
-F 3 "" H 7500 4700 50  0001 C CNN
-	1    7500 4700
-	0    -1   -1   0
-$EndComp
-Wire Wire Line
-	6850 4800 7550 4800
-Wire Wire Line
-	6850 5100 7550 5100
-Wire Wire Line
-	6850 5000 7550 5000
-Wire Wire Line
-	6850 4900 7550 4900
 Wire Wire Line
 	7150 3600 6850 3600
@@
 Wire Wire Line
 	8900 2300 8400 2300
-$Sheet
-S 850  3800 950  600
-U 5A7CD733
-F0 "MPU9250" 60
-F1 "MPU9250.sch" 60
-F2 "SCL" I R 1800 4000 60
-F3 "SDA" I R 1800 4100 60
-$EndSheet
-Wire Wire Line
-	7550 4700 7500 4700
-Wire Wire Line
-	1800 4000 2550 4000
 Wire Wire Line
 	2550 4000 2550 3950
 Connection ~ 2550 3950
 Wire Wire Line
-	1800 4100 2600 4100
-Wire Wire Line
 	2600 4100 2600 4050
 Connection ~ 2600 4050
-NoConn ~ 8350 5100
 Wire Wire Line
 	8900 1800 8400 1800
