File: Power.sch (KiCad schematic (older format))
At the start: 43 parts, among them J10 SUPPLY, J11 GND, J7 PH_A, J8 PH_B, J9 PH_C, Q1 IRF7749, Q2 IRF7749, Q3 IRF7749, Q4 IRF7749, Q5 IRF7749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

Commit message: removed HALL switch, added bulk capacitor, updated sheet's datestamp
Parts:
- added C50: 330uF_63V, Capacitors_THT:CP_Radial_D10.0mm_P5.00mm, symbol CP1
- C43, C44: value 680uF_63V -> 330uF_63V; footprint Capacitors_THT:CP_Radial_D12.5mm_P5.00mm -> Capacitors_THT:CP_Radial_D10.0mm_P5.00mm
Connections:
- net GND: now also C50.2
- net SUPPLY: now also C50.1
Other:
- note added: "UVZ1J331MPD x3"
